Commit message: xacro update for melodic

File: gazebo/gazebo.urdf.xacro (robot description, xacro)
@@ -10,4 +10,5 @@
        xmlns:controller="http://playerstage.sourceforge.net/gazebo/xmlschema/#controller"
        xmlns:interface="http://playerstage.sourceforge.net/gazebo/xmlschema/#interface"
+       xmlns:xacro="http://www.ros.org/wiki/xacro"
        name="pmb2">
   <gazebo>
@@ -68,4 +69,4 @@
   </gazebo>
   <!-- define global properties -->
-  <property name="M_PI" value="3.1415926535897931" />
+  <xacro:property name="M_PI" value="3.1415926535897931" />
 </robot>

File: robots/pmb2_custom.urdf.xacro (robot description, xacro)
@@ -11,5 +11,5 @@
         <!-- The properties below are modified using empy http://www.alcyone.com/software/empy/
              from the create_robot.py tool. Handle them with care -->
-   <property name="has_sonar" value="false"/>
+   <xacro:property name="has_sonar" value="false"/>
   <!-- The following included files set up definitions of parts of the robot body -->
   <!-- Base -->
@@ -21,6 +21,6 @@
   <!-- Now we can start using the macros included above to define the actual robot -->
   <xacro:base_sensors name="base" hokuyo="true" sonars="${has_sonar}" microphone="true" tof="true"/>
+  <xacro:include filename="$(find pmb2_description)/urdf/arm/arm.urdf.xacro"/>
   <xacro:include filename="$(find pmb2_description)/urdf/column/column.urdf.xacro" />
-  <xacro:include filename="$(find pmb2_description)/urdf/arm/arm.urdf.xacro" />
   <!--<xacro:ur5e_robot prefix="ur5e" />-->
 </robot>

File: urdf/base/base.urdf.xacro (robot description, xacro)
@@ -15,17 +15,17 @@
   <xacro:include filename="$(find pmb2_description)/urdf/objects/antenna.urdf.xacro"/>
   <!-- Wheel characteristics -->
-  <property name="wheel_radius"     value="0.0985"/>
-  <property name="wheel_width"      value="0.040"/>
-  <property name="wheel_separation" value="0.4044"/>
-  <property name="wheel_torque"     value="6.0"/>
-  <property name="wheel_velocity"   value="1.0"/>
+  <xacro:property name="wheel_radius"     value="0.0985"/>
+  <xacro:property name="wheel_width"      value="0.040"/>
+  <xacro:property name="wheel_separation" value="0.4044"/>
+  <xacro:property name="wheel_torque"     value="6.0"/>
+  <xacro:property name="wheel_velocity"   value="1.0"/>
   <!-- Caster wheel characteristics -->
-  <property name="caster_radius"       value="0.025"/>
-  <property name="caster_width"        value="0.015"/>
-  <property name="caster_separation_x" value="0.343"/>
-  <property name="caster_separation_y" value="0.204"/>
-  <property name="caster_offset_x"     value="-0.002"/>
-  <property name="caster_offset_y"     value="0.0"/>
-  <property name="caster_offset_z"     value="-0.0335"/>
+  <xacro:property name="caster_radius"       value="0.025"/>
+  <xacro:property name="caster_width"        value="0.015"/>
+  <xacro:property name="caster_separation_x" value="0.343"/>
+  <xacro:property name="caster_separation_y" value="0.204"/>
+  <xacro:property name="caster_offset_x"     value="-0.002"/>
+  <xacro:property name="caster_offset_y"     value="0.0"/>
+  <xacro:property name="caster_offset_z"     value="-0.0335"/>
   <xacro:macro name="base" params="name">
     <!-- Base -->

File: urdf/base/base_sensors.urdf.xacro (robot description, xacro)
@@ -18,7 +18,7 @@
   <xacro:include filename="$(find pmb2_description)/urdf/sensors/low_range_sensor.urdf.xacro"/>
   <!-- Laser characteristics -->
-  <property name="base_laser_x" value="0.202"/>
-  <property name="base_laser_y" value="0.0"/>
-  <property name="base_laser_z" value="-0.004"/>
+  <xacro:property name="base_laser_x" value="0.202"/>
+  <xacro:property name="base_laser_y" value="0.0"/>
+  <xacro:property name="base_laser_z" value="-0.004"/>
   <!--Modified by Sebastien ALTOUNIAN-->
   <!--<xacro:macro name="base_sensors" params=" name hokuyo:=false sick551:=false sick561:=false sick571:=false sonars:=false microphone:=false ">-->

File: urdf/objects/antenna.urdf.xacro (robot description, xacro)
@@ -39,5 +39,5 @@
       <parent link="${parent}"/>
       <child link="${name}_link"/>
-      <insert_block name="origin"/>
+      <xacro:insert_block name="origin"/>
     </joint>
   </xacro:macro>

File: urdf/sensors/low_range_sensor.urdf.xacro (robot description, xacro)
@@ -16,5 +16,5 @@
     </link>
     <joint name="${name}_joint" type="fixed">
-      <insert_block name="origin"/>
+      <xacro:insert_block name="origin"/>
       <axis xyz="0 0 0"/>
       <parent link="${parent}_link"/>
