Commit message: column 2023

File: urdf/column/column.urdf.xacro (robot description, xacro)
@@ -14,4 +14,48 @@
     </visual>
   </link>
+<link name="controlleur_ur5a">
+    <visual>
+      <geometry>
+        <box size="0.08 0.1 1.5"/>
+      </geometry>
+      <material name="grey">
+	      <color rgba="0.52 0.53 0.54 1.0"/>
+      </material>
+      <origin rpy="0 0 0" xyz="0 0 0.75"/>
+    </visual>
+  </link>
+<link name="jetson_n_power">
+    <visual>
+      <geometry>
+        <box size="0.06 0.06 1.5"/>
+      </geometry>
+      <material name="grey">
+	      <color rgba="0.52 0.53 0.54 1.0"/>
+      </material>
+      <origin rpy="0 0 0" xyz="0 0 0.75"/>
+    </visual>
+  </link>
+<link name="controlleur_back">
+    <visual>
+      <geometry>
+        <box size="0.16 0.16 1.5"/>
+      </geometry>
+      <material name="grey">
+	      <color rgba="0.52 0.53 0.54 1.0"/>
+      </material>
+      <origin rpy="0 0 0" xyz="0 0 0.75"/>
+    </visual>
+  </link>
+  <link name="AU">
+    <visual>
+      <geometry>
+        <box size="0.09 0.09 0.1"/>
+      </geometry>
+      <material name="grey">
+	      <color rgba="0.52 0.53 0.54 1.0"/>
+      </material>
+      <origin rpy="0 0 0" xyz="0 0 0.75"/>
+    </visual>
+  </link>
   <link name="vertical_cart">
     <visual>
@@ -25,4 +69,5 @@
     </visual>
   </link>
+<!--
   <link name="horizontal_arm">
     <visual>
@@ -36,4 +81,6 @@
     </visual>
   </link>
+-->
+  <!--
   <link name="arm_cylender">
     <visual>
@@ -58,4 +105,5 @@
     </visual>
   </link>
+   -->
   <link name="screen">
     <visual>
@@ -66,5 +114,5 @@
 	      <color rgba="0 0 0 1.0"/>
       </material>
-      <origin rpy="0 0 0" xyz="0 0 0"/>
+      <origin rpy="0 0 0" xyz="0 0.29 0"/>
     </visual>
   </link>
@@ -77,5 +125,5 @@
 	      <color rgba="0 0 0 1.0"/>
       </material>
-      <origin rpy="-0.3 0 0" xyz="0 0 0"/>
+      <origin xyz="0 0.26 0" rpy="-0.6457 0 0" />
     </visual>
   </link>
@@ -88,5 +136,5 @@
 	      <color rgba="0 0 0 1.0"/>
       </material>
-      <origin rpy="0.2 0 0" xyz="0 0 0"/>
+      <origin rpy="0.65 0 0" xyz="0 0 0"/>
     </visual>
   </link>
@@ -106,5 +154,25 @@
     <parent link="base_link"/>
     <child link="vertical_mast"/>
-    <origin xyz="0 0 0.2" rpy="0 0 -1.57"/>
+    <origin xyz="-0.07 0 0.2" rpy="0 0 -1.57"/>
+  </joint>
+  <joint name="joint_1b" type="fixed">
+    <parent link="vertical_mast"/>
+    <child link="controlleur_ur5a"/>
+    <origin xyz="0.1 0 0" rpy="0 0 0"/>
+  </joint>
+  <joint name="joint_back" type="fixed">
+    <parent link="vertical_mast"/>
+    <child link="controlleur_back"/>
+    <origin xyz="0 -0.08 0" rpy="0 0 0"/>
+  </joint>
+  <joint name="joint_1c" type="fixed">
+    <parent link="vertical_mast"/>
+    <child link="jetson_n_power"/>
+    <origin xyz="-0.07 0 0" rpy="0 0 0"/>
+  </joint>
+  <joint name="joint_1d" type="fixed">
+    <parent link="vertical_mast"/>
+    <child link="AU"/>
+    <origin xyz="-0.09 0 0" rpy="0 0 0"/>
   </joint>
   <joint name="joint_2" type="fixed">
@@ -116,24 +184,24 @@
     <limit lower="0.22" upper="1.2" effort="10" velocity="0.6"/> -->
   </joint>
-  <!--<joint name="joint_3" type="revolute">-->
+  <!--<joint name="joint_3" type="revolute">
   <joint name="joint_3" type="fixed">
     <parent link="vertical_cart"/>
     <child link="horizontal_arm"/>
     <origin xyz="0.12 0 0" rpy="0 0 0"/>
-    <!--<axis xyz="0 0 1" />
-    <limit lower="-1" upper="1" effort="10" velocity="0.8"/>-->
-  </joint>
+    <limit lower="-1" upper="1" effort="10" velocity="0.8"/>
+  </joint>-->
   <!--<joint name="joint_4" type="revolute">-->
+  <!--
   <joint name="joint_4" type="fixed">
     <parent link="horizontal_arm"/>
     <child link="arm_cylender"/>
     <origin xyz="0.24 0 0" rpy="3.14159 0 0"/>
-    <!--<axis xyz="1 0 0" />
-    <limit lower="0" upper="3" effort="10" velocity="0.8"/>-->
-  </joint>
+    <limit lower="0" upper="3" effort="10" velocity="0.8"/>
+  </joint>
+  -->
   <joint name="joint_5" type="fixed">
     <parent link="vertical_mast"/>
     <child link="screen"/>
-    <origin xyz="0 0.08 1.4" rpy="0 0 0"/>
+    <origin xyz="0 0 1.4" rpy="0 0 0"/>
   </joint>
   <joint name="joint_6" type="fixed">
@@ -145,6 +213,7 @@
     <parent link="vertical_mast"/>
     <child link="HRI_screen"/>
-    <origin xyz="-0.1 0.1 1" rpy="0 0 0"/>
-  </joint>
+    <origin xyz="0 0.24 1" rpy="0 0 0"/>
+  </joint>
+<!--
   <joint name="joint_8" type="fixed">
     <parent link="arm_cylender"/>
@@ -152,4 +221,5 @@
     <origin xyz="0 0 0" rpy="0 0 0"/>
   </joint>
+-->
  <xacro:sensor_d455 name="col_camera_sensor_d455" parent="vertical_mast" >
     <origin xyz="0 0 0" rpy="0 0 0"/>
@@ -158,5 +228,6 @@
     <parent link="vertical_mast"/>
     <child link="realsense_fake_link"/>
-    <origin xyz="0 0.22 0.92" rpy="-0.837758 0 0"/>
+    <origin xyz="0 0.27 0.92" rpy="-0.837758 0 0"/>
+    <!--<origin xyz="0 0.22 0.92" rpy="-0.837758 0 0"/>-->
   </joint>
   <link name="realsense_fake_link">
