Commit message: fix melodic warning

File: urdf/sensors/bumper.urdf.xacro (robot description, xacro)
@@ -35,5 +35,5 @@
     <joint name="${name}_joint" type="fixed">
       <axis xyz="0 1 0"/>
-      <xacro:insert_block name="origin"/>
+      <insert_block name="origin"/>
       <parent link="${parent}_link"/>
       <child  link="${name}_link"/>

File: urdf/sensors/hokuyo_urg_04lx_ug01_laser.urdf.xacro (robot description, xacro)
@@ -28,5 +28,5 @@
     <joint name="${name}_joint" type="fixed">
       <axis xyz="0 1 0"/>
-      <xacro:insert_block name="origin"/>
+      <insert_block name="origin"/>
       <parent link="${parent}_link"/>
       <child  link="${name}_link"/>

File: urdf/sensors/imu.urdf.xacro (robot description, xacro)
@@ -25,5 +25,5 @@
       <parent link="${parent}"/>
       <child link="${name}_link"/>
-      <xacro:insert_block name="origin"/>
+      <insert_block name="origin"/>
     </joint>
     <gazebo reference="${name}_link">

File: urdf/sensors/low_range_sensor.urdf.xacro (robot description, xacro)
@@ -16,5 +16,5 @@
     </link>
     <joint name="${name}_joint" type="fixed">
-      <xacro:insert_block name="origin"/>
+      <insert_block name="origin"/>
       <axis xyz="0 0 0"/>
       <parent link="${parent}_link"/>

File: urdf/sensors/microphone.urdf.xacro (robot description, xacro)
@@ -12,5 +12,5 @@
     <link name="${name}_link"/>
     <joint name="${name}_joint" type="fixed">
-      <xacro:insert_block name="origin"/>
+      <insert_block name="origin"/>
       <child link="${name}_link"/>
       <parent link="${parent}_link"/>

File: urdf/sensors/range.urdf.xacro (robot description, xacro)
@@ -27,5 +27,5 @@
     </link>
     <joint name="${name}_joint" type="fixed">
-      <xacro:insert_block name="origin"/>
+      <insert_block name="origin"/>
       <axis xyz="0 0 1"/>
       <parent link="${parent}_link"/>

File: urdf/sensors/realsense/realsense_D455_camera.urdf.xacro (robot description, xacro)
@@ -56,6 +56,6 @@
         <origin xyz="${d455_zero_depth_to_glass + d455_glass_to_front} ${-d455_cam_depth_py} 0" rpy="${M_PI/2} 0 ${M_PI/2}"/>
         <geometry>
-          <!-- <box size="${d455_cam_depth} ${d455_cam_width} ${d455_cam_height}"/> -->
-	        <mesh filename="package://realsense2_description/meshes/d455.stl" scale="0.001 0.001 0.001" />
+          <box size="${d455_cam_depth} ${d455_cam_width} ${d455_cam_height}"/>
+	        <!-- <mesh filename="package://realsense2_description/meshes/d455.stl" scale="0.001 0.001 0.001" /> -->
         </geometry>
         <material name="aluminum"/>

File: urdf/sensors/sick_tim551_laser.urdf.xacro (robot description, xacro)
@@ -28,5 +28,5 @@
     <joint name="${name}_joint" type="fixed">
       <axis xyz="0 1 0"/>
-      <xacro:insert_block name="origin"/>
+      <insert_block name="origin"/>
       <parent link="${parent}_link"/>
       <child  link="${name}_link"/>

File: urdf/sensors/sick_tim561_laser.urdf.xacro (robot description, xacro)
@@ -28,5 +28,5 @@
     <joint name="${name}_joint" type="fixed">
       <axis xyz="0 1 0"/>
-      <xacro:insert_block name="origin"/>
+      <insert_block name="origin"/>
       <parent link="${parent}_link"/>
       <child  link="${name}_link"/>

File: urdf/sensors/sick_tim571_laser.urdf.xacro (robot description, xacro)
@@ -28,5 +28,5 @@
     <joint name="${name}_joint" type="fixed">
       <axis xyz="0 1 0"/>
-      <xacro:insert_block name="origin"/>
+      <insert_block name="origin"/>
       <parent link="${parent}_link"/>
       <child  link="${name}_link"/>
